File: Universal-ISA-Backplane-Power.kicad_sch (KiCad schematic)
At the start: 23 parts, among them P101 ATX 20-Pin Power, P102 FRNT_PNL, Q101 BC547, U101 555, U102 7905

Commit message: Initial steps for PCB layout
Parts:
- added P103: HW_SW_PWR, Connector_PinHeader_2.54mm:PinHeader_1x02_P2.54mm_Vertical, symbol Connector_Generic:Conn_01x02
- P101: footprint Universal-ISA-Backplane:Molex_Mini-Fit_Jr_5569-20A2_2x10_P4.20mm_Horizontal -> Connector_Molex:Molex_Mini-Fit_Jr_5566-20A_2x10_P4.20mm_Vertical
- P102: value FRNT_PNL -> F_PANEL; footprint Connector_PinHeader_2.54mm:PinHeader_2x05_P2.54mm_Horizontal -> Connector_PinHeader_2.54mm:PinHeader_2x05_P2.54mm_Vertical
Connections:
- net PWR_SW1 is gone; now on an unnamed net: C101.1, R108.1, S101.2
- net PWR_SW2 is gone; now on an unnamed net: R106.2, R107.1, S101.1, U101.2 (TR), U101.6 (THR)
- net GND: now also P103.2 (Pin_2)
- net at P101.14 (~{PS_ON}), Q101.1 (C): now also P103.1 (Pin_1)
- no-connect marks 12 -> 10
Other:
- note added: "If using toggle switch for power (P103), these components do not fit."
Changed lines of the file:
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@@
   (junction (at 121.92 105.41) (diameter 0) (color 0 0 0 0)
   )
+  (junction (at 74.93 77.47) (diameter 0) (color 0 0 0 0)
+  )
   (junction (at 158.75 44.45) (diameter 0) (color 0 0 0 0)
   )
@@
   (junction (at 109.22 115.57) (diameter 0) (color 0 0 0 0)
   )
+  (junction (at 121.92 100.33) (diameter 0) (color 0 0 0 0)
+  )
   (junction (at 166.37 76.2) (diameter 0) (color 0 0 0 0)
   )
@@
   )
   (no_connect (at 100.33 95.25))
-  (no_connect (at 110.49 54.61))
-  (no_connect (at 97.79 57.15))
-  (no_connect (at 97.79 59.69))
-  (no_connect (at 97.79 62.23))
-  (no_connect (at 97.79 64.77))
-  (no_connect (at 110.49 64.77))
-  (no_connect (at 110.49 62.23))
-  (no_connect (at 110.49 59.69))
-  (no_connect (at 110.49 57.15))
+  (no_connect (at 162.56 69.85))
+  (no_connect (at 149.86 77.47))
+  (no_connect (at 149.86 80.01))
+  (no_connect (at 162.56 80.01))
+  (no_connect (at 162.56 77.47))
+  (no_connect (at 162.56 74.93))
+  (no_connect (at 162.56 72.39))
   (no_connect (at 196.85 59.69))
   (no_connect (at 171.45 59.69))
@@
     (stroke (width 0) (type default) (color 0 0 0 0))
   )
+  (wire (pts (xy 74.93 77.47) (xy 74.93 95.25))
+    (stroke (width 0) (type default) (color 0 0 0 0))
+  )
   (wire (pts (xy 158.75 44.45) (xy 168.91 44.45))
     (stroke (width 0) (type default) (color 0 0 0 0))
@@
     (stroke (width 0) (type default) (color 0 0 0 0))
   )
-  (wire (pts (xy 74.93 38.1) (xy 74.93 95.25))
+  (wire (pts (xy 74.93 38.1) (xy 74.93 77.47))
     (stroke (width 0) (type default) (color 0 0 0 0))
   )
@@
     (stroke (width 0) (type default) (color 0 0 0 0))
   )
-  (wire (pts (xy 147.32 100.33) (xy 147.32 44.45))
+  (wire (pts (xy 121.92 100.33) (xy 121.92 44.45))
     (stroke (width 0) (type default) (color 0 0 0 0))
   )
@@
     (stroke (width 0) (type default) (color 0 0 0 0))
   )
+  (wire (pts (xy 148.59 91.44) (xy 148.59 74.93))
+    (stroke (width 0) (type default) (color 0 0 0 0))
+  )
   (wire (pts (xy 195.58 82.55) (xy 196.85 82.55))
     (stroke (width 0) (type default) (color 0 0 0 0))
@@
     (stroke (width 0) (type default) (color 0 0 0 0))
   )
+  (wire (pts (xy 146.05 93.98) (xy 196.85 93.98))
+    (stroke (width 0) (type default) (color 0 0 0 0))
+  )
+  (wire (pts (xy 146.05 72.39) (xy 149.86 72.39))
+    (stroke (width 0) (type default) (color 0 0 0 0))
+  )
   (wire (pts (xy 173.99 127) (xy 180.34 127))
     (stroke (width 0) (type default) (color 0 0 0 0))
@@
     (stroke (width 0) (type default) (color 0 0 0 0))
   )
-  (wire (pts (xy 184.15 87.63) (xy 172.72 87.63))
-    (stroke (width 0) (type default) (color 0 0 0 0))
-  )
-  (wire (pts (xy 196.85 82.55) (xy 196.85 91.44))
+  (wire (pts (xy 74.93 77.47) (xy 78.74 77.47))
+    (stroke (width 0) (type default) (color 0 0 0 0))
+  )
+  (wire (pts (xy 148.59 91.44) (xy 184.15 91.44))
+    (stroke (width 0) (type default) (color 0 0 0 0))
+  )
+  (wire (pts (xy 148.59 74.93) (xy 149.86 74.93))
+    (stroke (width 0) (type default) (color 0 0 0 0))
+  )
+  (wire (pts (xy 196.85 82.55) (xy 196.85 93.98))
     (stroke (width 0) (type default) (color 0 0 0 0))
   )
@@
     (stroke (width 0) (type default) (color 0 0 0 0))
   )
-  (wire (pts (xy 100.33 100.33) (xy 147.32 100.33))
+  (wire (pts (xy 100.33 100.33) (xy 121.92 100.33))
     (stroke (width 0) (type default) (color 0 0 0 0))
   )
@@
     (stroke (width 0) (type default) (color 0 0 0 0))
   )
-  (wire (pts (xy 147.32 44.45) (xy 158.75 44.45))
+  (wire (pts (xy 121.92 44.45) (xy 158.75 44.45))
     (stroke (width 0) (type default) (color 0 0 0 0))
   )
@@
     (stroke (width 0) (type default) (color 0 0 0 0))
   )
-  (wire (pts (xy 172.72 91.44) (xy 196.85 91.44))
-    (stroke (width 0) (type default) (color 0 0 0 0))
-  )
-  (wire (pts (xy 184.15 82.55) (xy 184.15 87.63))
+  (wire (pts (xy 184.15 82.55) (xy 184.15 91.44))
+    (stroke (width 0) (type default) (color 0 0 0 0))
+  )
+  (polyline (pts (xy 135.89 31.75) (xy 233.68 31.75))
     (stroke (width 0) (type default) (color 0 0 0 0))
   )
@@
     (stroke (width 0) (type default) (color 0 0 0 0))
   )
+  (wire (pts (xy 121.92 100.33) (xy 147.32 100.33))
+    (stroke (width 0) (type default) (color 0 0 0 0))
+  )
   (wire (pts (xy 190.5 44.45) (xy 184.15 44.45))
     (stroke (width 0) (type default) (color 0 0 0 0))
   )
+  (polyline (pts (xy 233.68 31.75) (xy 233.68 96.52))
+    (stroke (width 0) (type default) (color 0 0 0 0))
+  )
+  (polyline (pts (xy 233.68 96.52) (xy 135.89 96.52))
+    (stroke (width 0) (type default) (color 0 0 0 0))
+  )
   (wire (pts (xy 223.52 38.1) (xy 74.93 38.1))
     (stroke (width 0) (type default) (color 0 0 0 0))
@@
     (stroke (width 0) (type default) (color 0 0 0 0))
   )
+  (wire (pts (xy 146.05 93.98) (xy 146.05 72.39))
+    (stroke (width 0) (type default) (color 0 0 0 0))
+  )
   (wire (pts (xy 185.42 82.55) (xy 184.15 82.55))
     (stroke (width 0) (type default) (color 0 0 0 0))
   )
+  (polyline (pts (xy 135.89 31.75) (xy 135.89 96.52))
+    (stroke (width 0) (type default) (color 0 0 0 0))
+  )
   (wire (pts (xy 156.21 115.57) (xy 191.77 115.57))
     (stroke (width 0) (type default) (color 0 0 0 0))
@@
     (stroke (width 0) (type default) (color 0 0 0 0))
   )
-  (text "ATX Power On" (at 180.34 34.29 0)
+  (text "If using toggle switch for power (P103), these components do not fit."
+    (at 135.89 30.48 0)
     (effects (font (size 1.27 1.27)) (justify left bottom))
   )
-  (label "PWR_SW2" (at 172.72 87.63 0)
-    (effects (font (size 1.27 1.27)) (justify left bottom))
-  )
-  (label "PWR_SW1" (at 172.72 91.44 0)
+  (text "ATX Power On" (at 180.34 36.83 0)
     (effects (font (size 1.27 1.27)) (justify left bottom))
   )
@@
       (effects (font (size 1.524 1.524)))
     )
-    (property "Footprint" "Universal-ISA-Backplane:Molex_Mini-Fit_Jr_5569-20A2_2x10_P4.20mm_Horizontal" (id 2) (at 87.63 107.95 0)
+    (property "Footprint" "Connector_Molex:Molex_Mini-Fit_Jr_5566-20A_2x10_P4.20mm_Vertical" (id 2) (at 87.63 107.95 0)
       (effects (font (size 1.27 1.27)) hide)
     )
@@
     (pin "1")
   )
+  (symbol (lib_id "power:GND") (at 78.74 80.01 0) (unit 1)
+    (in_bom yes) (on_board yes) (fields_autoplaced)
+    (property "Reference" "#PWR03" (id 0) (at 78.74 86.36 0)
+      (effects (font (size 1.27 1.27)) hide)
+    )
+    (property "Value" "GND" (id 1) (at 78.74 85.09 0)
+      (effects (font (size 1.27 1.27)) hide)
+    )
+    (property "Footprint" "" (id 2) (at 78.74 80.01 0)
+      (effects (font (size 1.27 1.27)) hide)
+    )
+    (property "Datasheet" "" (id 3) (at 78.74 80.01 0)
+      (effects (font (size 1.27 1.27)) hide)
+    )
+    (pin "1")
+  )
   (symbol (lib_id "Device:C") (at 194.31 44.45 90) (unit 1)
     (in_bom yes) (on_board yes)
@@
     (pin "1")
   )
-  (symbol (lib_id "Universal-ISA-Backplane-symbols:Conn_2Rows-09Pins") (at 105.41 59.69 180) (unit 1)
-    (in_bom yes) (on_board yes)
-    (property "Reference" "P102" (id 0) (at 104.14 48.895 0))
-    (property "Value" "FRNT_PNL" (id 1) (at 104.14 51.2064 0))
-    (property "Footprint" "Connector_PinHeader_2.54mm:PinHeader_2x05_P2.54mm_Horizontal" (id 2) (at 105.41 59.69 0)
-      (effects (font (size 1.27 1.27)) hide)
-    )
-    (property "Datasheet" "~" (id 3) (at 105.41 59.69 0)
-      (effects (font (size 1.27 1.27)) hide)
-    )
-    (pin "1")
+  (symbol (lib_id "Universal-ISA-Backplane-symbols:Conn_2Rows-09Pins") (at 157.48 74.93 180) (unit 1)
+    (in_bom yes) (on_board yes)
+    (property "Reference" "P102" (id 0) (at 156.21 84.8614 0))
+    (property "Value" "F_PANEL" (id 1) (at 156.21 82.55 0))
+    (property "Footprint" "Connector_PinHeader_2.54mm:PinHeader_2x05_P2.54mm_Vertical" (id 2) (at 157.48 74.93 0)
+      (effects (font (size 1.27 1.27)) hide)
+    )
+    (property "Datasheet" "~" (id 3) (at 157.48 74.93 0)
+      (effects (font (size 1.27 1.27)) hide)
+    )
+    (pin "1")
+    (pin "10")
     (pin "2")
     (pin "3")
@@
     (pin "9")
   )
+  (symbol (lib_id "Connector_Generic:Conn_01x02") (at 83.82 77.47 0) (unit 1)
+    (in_bom yes) (on_board yes) (fields_autoplaced)
+    (property "Reference" "P103" (id 0) (at 86.36 77.4699 0)
+      (effects (font (size 1.27 1.27)) (justify left))
+    )
+    (property "Value" "HW_SW_PWR" (id 1) (at 86.36 80.0099 0)
+      (effects (font (size 1.27 1.27)) (justify left))
+    )
+    (property "Footprint" "Connector_PinHeader_2.54mm:PinHeader_1x02_P2.54mm_Vertical" (id 2) (at 83.82 77.47 0)
+      (effects (font (size 1.27 1.27)) hide)
+    )
+    (property "Datasheet" "~" (id 3) (at 83.82 77.47 0)
+      (effects (font (size 1.27 1.27)) hide)
+    )
+    (pin "1")
+    (pin "2")
+  )
   (sheet_instances

Commit message: PC/104 and ISA connector fixes
And further development
Changed lines of the file:
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@@
-    (stroke (width 0) (type default) (color 0 0 0 0))
-  )
-  (polyline (pts (xy 135.89 31.75) (xy 233.68 31.75))
     (stroke (width 0) (type default) (color 0 0 0 0))
   )
@@
     (stroke (width 0) (type default) (color 0 0 0 0))
   )
-  (polyline (pts (xy 233.68 31.75) (xy 233.68 96.52))
-    (stroke (width 0) (type default) (color 0 0 0 0))
-  )
-  (polyline (pts (xy 233.68 96.52) (xy 135.89 96.52))
-    (stroke (width 0) (type default) (color 0 0 0 0))
-  )
   (wire (pts (xy 223.52 38.1) (xy 74.93 38.1))
     (stroke (width 0) (type default) (color 0 0 0 0))
@@
   )
   (wire (pts (xy 185.42 82.55) (xy 184.15 82.55))
-    (stroke (width 0) (type default) (color 0 0 0 0))
-  )
-  (polyline (pts (xy 135.89 31.75) (xy 135.89 96.52))
     (stroke (width 0) (type default) (color 0 0 0 0))
   )
@@
     )
     (pin "1")
-    (pin "10")
     (pin "2")
     (pin "3")
