File: Universal-ISA-Backplane.kicad_pcb (KiCad board)
At the start: 4 copper layers, 0 parts

Commit message: Initial steps for PCB layout
Parts:
- added C101: µ47 10% 50V CR X7R, Capacitor_THT:C_Disc_D6.0mm_W4.4mm_P5.00mm, F.Cu at (112.5, 179.0)
- added C102: µ1 10% 50V CR X7R, Capacitor_THT:C_Disc_D6.0mm_W4.4mm_P5.00mm, F.Cu at (120.4, 200.2)
- added CR101: +5VSB, LED_THT:LED_D3.0mm, F.Cu at (178.8, 215.9)
- added CR102: +5V, LED_THT:LED_D3.0mm, F.Cu at (186.7, 215.9)
- added CR103: +12V, LED_THT:LED_D3.0mm, F.Cu at (170.4, 215.9)
- added CR104: -12V, LED_THT:LED_D3.0mm, F.Cu at (194.8, 213.4)
- added CR105: -5V, LED_THT:LED_D3.0mm, F.Cu at (162.6, 213.4)
- added ITEM1: Heatsink_Pad, Heatsink:Heatsink_Fischer_SK104-STC-STIC_35x13mm_2xDrill2.5mm, F.Cu at (260.4, 185.9)
- added P101: ATX 20-Pin Power, Connector_Molex:Molex_Mini-Fit_Jr_5566-20A_2x10_P4.20mm_Vertical, F.Cu at (206.9, 216.2)
- added P102: F_PANEL, Connector_PinHeader_2.54mm:PinHeader_2x05_P2.54mm_Vertical, F.Cu at (142.2, 220.7)
- added P103: HW_SW_PWR, Connector_PinHeader_2.54mm:PinHeader_1x02_P2.54mm_Vertical, F.Cu at (133.6, 220.7)
- added P201: PC104, Universal-ISA-Backplane:PC104_Platform, F.Cu at (237.7, 142.1)
- added Q101: BC547, Package_TO_SOT_THT:TO-92_Inline, F.Cu at (109.5, 204.1)
- added R101: 270R 10% QW MF, Resistor_THT:R_Axial_DIN0204_L3.6mm_D1.6mm_P5.08mm_Horizontal, F.Cu at (178.8, 218.4)
- added R102: 270R 10% QW MF, Resistor_THT:R_Axial_DIN0204_L3.6mm_D1.6mm_P5.08mm_Horizontal, F.Cu at (186.7, 223.5)
- added R103: 1K 10% QW MF, Resistor_THT:R_Axial_DIN0204_L3.6mm_D1.6mm_P5.08mm_Horizontal, F.Cu at (170.4, 223.5)
- added R104: 1K 10% QW MF, Resistor_THT:R_Axial_DIN0204_L3.6mm_D1.6mm_P5.08mm_Horizontal, F.Cu at (194.8, 223.5)
- added R105: 270R 10% QW MF, Resistor_THT:R_Axial_DIN0204_L3.6mm_D1.6mm_P5.08mm_Horizontal, F.Cu at (162.6, 223.5)
- added R106: 100K 10% QW MF, Resistor_THT:R_Axial_DIN0204_L3.6mm_D1.6mm_P5.08mm_Horizontal, F.Cu at (135.9, 174.5)
- added R107: 100K 10% QW MF, Resistor_THT:R_Axial_DIN0204_L3.6mm_D1.6mm_P5.08mm_Horizontal, F.Cu at (121.2, 168.7)
- added R108: 270K 10% QW MF, Resistor_THT:R_Axial_DIN0204_L3.6mm_D1.6mm_P5.08mm_Horizontal, F.Cu at (108.2, 184.4)
- added R109: 100K 10% QW MF, Resistor_THT:R_Axial_DIN0204_L3.6mm_D1.6mm_P5.08mm_Horizontal, F.Cu at (108.2, 192.0)
- added S101: Power, Button_Switch_THT:SW_PUSH_6mm, F.Cu at (120.6, 174.5)
- added U101: 555, Package_DIP:DIP-8_W7.62mm, F.Cu at (120.4, 185.4)
- added U102: 7905, Package_TO_SOT_THT:TO-220-3_Vertical, F.Cu at (255.5, 183.4)
Routing:
- net /Power/+5VSB: track 0.00 -> 202.9 mm, vias 0 -> 1
- net /ISA1/-5V: track 0.00 -> 155.2 mm, vias 0 -> 2
- net /ISA1/+12V: track 0.00 -> 149.2 mm, vias 0 -> 2
- net Net-(P101-Pad14): track 0.00 -> 139.2 mm
- net /ISA1/-12V: track 0.00 -> 99.2 mm
- net Net-(P102-Pad6): track 0.00 -> 87.9 mm
- net Net-(C101-Pad1): track 0.00 -> 83.1 mm
- net /ISA1/+5V: track 0.00 -> 76.3 mm
- net Net-(R108-Pad2): track 0.00 -> 15.2 mm
- net Net-(P101-Pad1): track 0.00 -> 9.70 mm
- net Net-(Q101-Pad2): track 0.00 -> 7.01 mm
- net Net-(CR105-Pad2): track 0.00 -> 2.54 mm
- net Net-(CR104-Pad2): track 0.00 -> 2.54 mm
- net Net-(CR103-Pad1): track 0.00 -> 2.54 mm
- net Net-(CR102-Pad1): track 0.00 -> 2.54 mm
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- added copper zone on B.Cu, net GND
- added copper zone on F.Cu, net GND
Other:
- board outline added: 243.8 x 243.8 mm

Commit message: PC/104 and ISA connector fixes
And further development
Parts:
- added H1: MountingHole_Pad, MountingHole:MountingHole_4mm_Pad_TopBottom, F.Cu at (72.8, 35.2)
- added H2: MountingHole_Pad, MountingHole:MountingHole_4mm_Pad_TopBottom, F.Cu at (118.5, 35.2)
- added H3: MountingHole_Pad, MountingHole:MountingHole_4mm_Pad_TopBottom, F.Cu at (276.0, 58.0)
- added H4: MountingHole_Pad, MountingHole:MountingHole_4mm_Pad_TopBottom, F.Cu at (118.5, 190.1)
- added H5: MountingHole_Pad, MountingHole:MountingHole_4mm_Pad_TopBottom, F.Cu at (276.0, 190.1)
- added H6: MountingHole_Pad, MountingHole:MountingHole_4mm_Pad_TopBottom, F.Cu at (118.5, 262.5)
- added H7: MountingHole_Pad, MountingHole:MountingHole_4mm_Pad_TopBottom, F.Cu at (276.0, 262.5)
- added H8: MountingHole_Pad, MountingHole:MountingHole_4mm_Pad_TopBottom, F.Cu at (52.5, 190.1)
- added H9: MountingHole_Pad, MountingHole:MountingHole_4mm_Pad_TopBottom, F.Cu at (72.8, 190.1)
- added J301: Bus_ISA_16bit, Universal-ISA-Backplane:ISA16, F.Cu at (42.8, 118.2)
- moved P201 107.7 mm to (164.1, 63.5), turned to 180 degrees
- moved C102 35.2 mm to (97.3, 226.6)
- moved R106 35.2 mm to (112.7, 201.0)
- moved P102 35.2 mm to (119.1, 247.2)
- moved C101 35.2 mm to (89.4, 205.5)
- moved R107 35.2 mm to (98.0, 195.1)
- moved R108 35.2 mm to (85.0, 210.9)
- moved R109 35.2 mm to (85.0, 218.5)
- moved S101 35.2 mm to (97.5, 201.0)
- moved U101 35.2 mm to (97.2, 211.9)
- moved P103 35.2 mm to (110.4, 247.2)
- moved Q101 35.2 mm to (86.3, 230.6)
- moved CR104 28.2 mm to (185.2, 239.9)
- moved ITEM1 28.2 mm to (250.8, 212.4)
- moved R104 28.2 mm to (185.2, 250.0)
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Connections:
- P102 pad 10: unconnected-(P102-Pad10) -> (no net)
Routing:
- net /Power/+5VSB: track 202.9 -> 20.7 mm, vias 1 -> 0
- net /ISA1/-5V: track 155.2 -> 0.00 mm, vias 2 -> 0
- net /ISA1/+12V: track 149.2 -> 0.00 mm, vias 2 -> 0
- net Net-(P101-Pad14): track 139.2 -> 0.00 mm
- net /ISA1/-12V: track 99.2 -> 0.00 mm
- net /ISA1/+5V: track 76.3 -> 0.00 mm
- net Net-(C101-Pad1): track 83.1 -> 21.8 mm
- net Net-(P101-Pad1): track 9.70 -> 0.00 mm
